File: kabeltester/hardware/kicad/kanalkarte/kanalkarte.kicad_pcb (KiCad board)
At the start: 4 copper layers, 118 x 74 mm, 413 parts, among them J1 DIN 41612 C96 Feder, J2 Messkarte, U1 SN74HC595PW, U10 CD74HCT4067M96, U11 ADG1606BRUZ, U12 CD74HCT4067M96, U13 ADG1606BRUZ, U14 CD74HCT4067M96, U15 ADG1606BRUZ, U16 CD74HCT4067M96, U17 ADG1606BRUZ, U18 CD74HCT4067M96, U2 SN74HC595PW, U3 ADG1606BRUZ, U4 CD74HCT4067M96, U5 ADG1606BRUZ, U6 CD74HCT4067M96, U7 ADG1606BRUZ, U8 CD74HCT4067M96, U9 ADG1606BRUZ

Commit message: Kanalkarte: ungerouteter Stand (Routing nach Container-Neustart neu gestartet)
Co-Authored-By: Claude Opus 5.5 <noreply@anthropic.com>
Claude-Session: https://claude.ai/code/session_0119zGeGQCWTR3UwpEi96iWe
Routing:
- added copper zone on In2.Cu, net 5VA
Changed lines of the file:
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@@
   (layers
     (0 "F.Cu" signal)
-    (1 "In1.Cu" power)
+    (1 "In1.Cu" signal)
     (2 "In2.Cu" signal)
     (31 "B.Cu" signal)
@@
   )
   (zone (net 149) (net_name "GND") (layer "F.Cu") (hatch edge 0.5)
-    (connect_pads yes (clearance 0.2))
+    (connect_pads (clearance 0.25))
     (min_thickness 0.2) (filled_areas_thickness no)
     (fill yes (thermal_gap 0.3) (thermal_bridge_width 0.35))
@@
   )
   (zone (net 149) (net_name "GND") (layer "In1.Cu") (hatch edge 0.5)
-    (connect_pads yes (clearance 0.2))
+    (connect_pads (clearance 0.25))
+    (min_thickness 0.2) (filled_areas_thickness no)
+    (fill yes (thermal_gap 0.3) (thermal_bridge_width 0.35))
+    (polygon
+      (pts
+        (xy 0.4 0.4)
+        (xy 117.6 0.4)
+        (xy 117.6 73.6)
+        (xy 0.4 73.6)
+      )
+    )
+  )
+  (zone (net 3) (net_name "5VA") (layer "In2.Cu") (hatch edge 0.5)
+    (connect_pads (clearance 0.25))
     (min_thickness 0.2) (filled_areas_thickness no)
     (fill yes (thermal_gap 0.3) (thermal_bridge_width 0.35))
@@
   )
   (zone (net 149) (net_name "GND") (layer "B.Cu") (hatch edge 0.5)
-    (connect_pads yes (clearance 0.2))
+    (connect_pads (clearance 0.25))
     (min_thickness 0.2) (filled_areas_thickness no)
     (fill yes (thermal_gap 0.3) (thermal_bridge_width 0.35))

Commit message: Zwischenstand: Messkarte/Kanalkarte während des Routings (wird ersetzt)
Co-Authored-By: Claude Opus 5.5 <noreply@anthropic.com>
Claude-Session: https://claude.ai/code/session_0119zGeGQCWTR3UwpEi96iWe
Routing:
- removed copper zone on In2.Cu, net 5VA
Changed lines of the file:
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@@
   (layers
     (0 "F.Cu" signal)
-    (1 "In1.Cu" signal)
+    (1 "In1.Cu" power)
     (2 "In2.Cu" signal)
     (31 "B.Cu" signal)
@@
   )
   (zone (net 149) (net_name "GND") (layer "F.Cu") (hatch edge 0.5)
-    (connect_pads (clearance 0.25))
+    (connect_pads yes (clearance 0.2))
     (min_thickness 0.2) (filled_areas_thickness no)
     (fill yes (thermal_gap 0.3) (thermal_bridge_width 0.35))
@@
   )
   (zone (net 149) (net_name "GND") (layer "In1.Cu") (hatch edge 0.5)
-    (connect_pads (clearance 0.25))
-    (min_thickness 0.2) (filled_areas_thickness no)
-    (fill yes (thermal_gap 0.3) (thermal_bridge_width 0.35))
-    (polygon
-      (pts
-        (xy 0.4 0.4)
-        (xy 117.6 0.4)
-        (xy 117.6 73.6)
-        (xy 0.4 73.6)
-      )
-    )
-  )
-  (zone (net 3) (net_name "5VA") (layer "In2.Cu") (hatch edge 0.5)
-    (connect_pads (clearance 0.25))
+    (connect_pads yes (clearance 0.2))
     (min_thickness 0.2) (filled_areas_thickness no)
     (fill yes (thermal_gap 0.3) (thermal_bridge_width 0.35))
@@
   )
   (zone (net 149) (net_name "GND") (layer "B.Cu") (hatch edge 0.5)
-    (connect_pads (clearance 0.25))
+    (connect_pads yes (clearance 0.2))
     (min_thickness 0.2) (filled_areas_thickness no)
     (fill yes (thermal_gap 0.3) (thermal_bridge_width 0.35))
