File: kabeltester/hardware/kicad/adapter_rj45/adapter_rj45.kicad_sch (KiCad schematic)
At the start: 7 parts, among them J1 DIN 41612 C96 Messer, J2 RJ45 Port 1, J3 RJ45 Port 2, U1 24AA02T-I/OT

Commit message: Adapter-Platine vollständig geroutet (DRC 0 Fehler), SES-Import und Masse-Vias im Generator
- routen.py: Freerouting auf vorhandener Platine, eigener SES-Import (KiCad 7 kann das in Python nicht)
- Masseflächen mit voller Anbindung, Masse-Durchkontaktierungen im Raster
- Adapter: Reservepins b9/b10 unbeschaltet (zweilagig nicht anbindbar)

Co-Authored-By: Claude Opus 5.5 <noreply@anthropic.com>
Claude-Session: https://claude.ai/code/session_0119zGeGQCWTR3UwpEi96iWe
Connections:
- net GND: no longer J1.b10, J1.b9
- no-connect marks 69 -> 71
Changed lines of the file:
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@@
     (instances
       (project "adapter_rj45"
-        (path "/67c804fc-43a7-4ad6-9edb-0d2313e90c63"
+        (path "/69fcb4cd-76d0-464f-9d5d-0028c03b5c50"
           (reference "J1")
           (unit 1)))))
@@
       (justify right bottom))
 )
-  (label "GND"
-    (at 31.75 139.7 180)
-    (fields_autoplaced)
-    (effects
-      (font
-        (size 1.27 1.27))
-      (justify right bottom))
-)
-  (label "GND"
-    (at 31.75 142.24 180)
-    (fields_autoplaced)
-    (effects
-      (font
-        (size 1.27 1.27))
-      (justify right bottom))
+  (no_connect
+    (at 31.75 139.7)
+)
+  (no_connect
+    (at 31.75 142.24)
 )
   (no_connect
@@
     (instances
       (project "adapter_rj45"
-        (path "/67c804fc-43a7-4ad6-9edb-0d2313e90c63"
+        (path "/69fcb4cd-76d0-464f-9d5d-0028c03b5c50"
           (reference "J2")
           (unit 1)))))
@@
     (instances
       (project "adapter_rj45"
-        (path "/67c804fc-43a7-4ad6-9edb-0d2313e90c63"
+        (path "/69fcb4cd-76d0-464f-9d5d-0028c03b5c50"
           (reference "J3")
           (unit 1)))))
@@
     (instances
       (project "adapter_rj45"
-        (path "/67c804fc-43a7-4ad6-9edb-0d2313e90c63"
+        (path "/69fcb4cd-76d0-464f-9d5d-0028c03b5c50"
           (reference "U1")
           (unit 1)))))
@@
     (instances
       (project "adapter_rj45"
-        (path "/67c804fc-43a7-4ad6-9edb-0d2313e90c63"
+        (path "/69fcb4cd-76d0-464f-9d5d-0028c03b5c50"
           (reference "C1")
           (unit 1)))))
@@
     (instances
       (project "adapter_rj45"
-        (path "/67c804fc-43a7-4ad6-9edb-0d2313e90c63"
+        (path "/69fcb4cd-76d0-464f-9d5d-0028c03b5c50"
           (reference "H1")
           (unit 1)))))
@@
     (instances
       (project "adapter_rj45"
-        (path "/67c804fc-43a7-4ad6-9edb-0d2313e90c63"
+        (path "/69fcb4cd-76d0-464f-9d5d-0028c03b5c50"
           (reference "H2")
           (unit 1)))))
